Commit message: Refactor multi_robot_arm package for Gazebo Harmonic simulation support
- Updated CMakeLists.txt to replace gazebo_ros with ros_gz_sim and added installation of Python scripts.
- Modified ros_controllers_robot.yaml to remove gripper controller parameters.
- Enhanced gazebo_arm.launch.py to use xacro for loading YAML files.
- Created new launch file for Gazebo Harmonic simulation.
- Updated package.xml to reflect version change and new dependencies.
- Added new Python scripts for pose goals and continuous waving/dance like motion.
- Refined URDF and Xacro files for compatibility with new simulation framework.
- Created empty SDF and updated empty.world for improved lighting and physics.
- Add demo video and update README for ROS2 Jazzy and Gazebo Harmonic support

File: urdf/ur/ur5/ur_ros2_control.xacro (robot description, xacro)
@@ -20,8 +20,8 @@
       <hardware>
         <xacro:if value="${sim_gazebo}">
-          <plugin>gazebo_ros2_control/GazeboSystem</plugin>
+          <plugin>gz_ros2_control/GazeboSimSystem</plugin>
         </xacro:if>
         <xacro:if value="${sim_ignition}">
-          <plugin>ign_ros2_control/IgnitionSystem</plugin>
+          <plugin>gz_ros2_control/GazeboSimSystem</plugin>
         </xacro:if>
         <xacro:if value="${use_fake_hardware}">
@@ -150,14 +150,4 @@
         <state_interface name="velocity"/>
         <state_interface name="effort"/>
-      </joint>
-      <joint name="${prefix}gripper_joint1">
-        <command_interface name="position"/>
-        <state_interface name="position">
-        <param name="initial_value">0</param>
-        </state_interface>
-      </joint>
-      <joint name="${prefix}gripper_joint2">
-        <command_interface name="position"/>
-        <state_interface name="position"/>
       </joint>
       <xacro:unless value="${sim_gazebo or sim_ignition}">

File: urdf/ur/ur5/ur_urdf.xacro (robot description, xacro)
@@ -66,5 +66,5 @@
      sim_ignition="$(arg sim_ignition)"
      headless_mode="$(arg headless_mode)"
-     initial_positions="${load_yaml(initial_positions_file)}"
+     initial_positions="${xacro.load_yaml(initial_positions_file)}"
      use_tool_communication="$(arg use_tool_communication)"
      tool_voltage="$(arg tool_voltage)"
@@ -122,5 +122,5 @@
       </joint>
       <gazebo>
-        <plugin filename="libgazebo_ros2_control.so" name="gazebo_ros2_control">
+        <plugin filename="libgz_ros2_control-system.so" name="gz_ros2_control::GazeboSimROS2ControlPlugin">
           <ros>
             <namespace>$(arg namespace)</namespace>
@@ -135,5 +135,5 @@
     </gazebo>
     <gazebo>
-      <plugin filename="libign_ros2_control-system.so" name="ign_ros2_control::IgnitionROS2ControlPlugin">
+      <plugin filename="libgz_ros2_control-system.so" name="gz_ros2_control::GazeboSimROS2ControlPlugin">
         <parameters>$(arg simulation_controllers)</parameters>
         <controller_manager_node_name>$(arg prefix)controller_manager</controller_manager_node_name>
